Commit message: updated for new rubric

File: src/slam_project/urdf/circle_bot_depth.xacro (robot description, xacro)
@@ -10,8 +10,15 @@
   <joint type="fixed" name="camera_joint">
     <origin xyz="0.2 0 0" rpy="0 0 0"/>
-    <child link="camera"/>
+    <child link="camera_link"/>
     <parent link="chassis"/>
   </joint>
- <link name='camera'>
+  <joint name="camera_optical_joint" type="fixed">
+    <origin xyz="0 0 0" rpy="-1.5707 0 -1.5707"/>
+    <parent link="camera_link"/>
+    <child link="camera_link_optical"/>
+  </joint>
+  <link name="camera_link_optical">
+  </link>
+ <link name='camera_link'>
     <inertial>
       <mass value="0.56"/>
